File: hardware/caravel_breakout_sstl/caravel_breakout_sstl.kicad_sch (KiCad schematic)
At the start: 33 parts, among them J1 Conn_02x07_Top_Bottom, J2 Conn_Coaxial, J3 Conn_02x07_Top_Bottom, J4 Conn_02x07_Top_Bottom, T1 Logo, T2 Logo, U1 Caravel, U2 LTC1844ES5-1.5, U3 SN74AVC4T245PW, U4 SN74AVC4T245PW

Commit message: Minor updates to improve routing
Ground all unused pins
Connections:
- net GND: now also J1.11 (Pin_11), J3.1 (Pin_1), J3.11 (Pin_11), J3.13 (Pin_13), J3.3 (Pin_3), J3.5 (Pin_5), J3.7 (Pin_7), J3.9 (Pin_9)
- net vccd: no longer J1.11 (Pin_11)
- no-connect marks 29 -> 22
Changed lines of the file:
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@@
   (no_connect (at 41.91 52.07))
   (no_connect (at 41.91 57.15))
-  (no_connect (at 252.73 121.92))
-  (no_connect (at 252.73 116.84))
-  (no_connect (at 252.73 119.38))
-  (no_connect (at 252.73 132.08))
-  (no_connect (at 252.73 129.54))
-  (no_connect (at 252.73 127))
-  (no_connect (at 252.73 124.46))
   (wire (pts (xy 129.54 64.77) (xy 125.73 64.77))
     (stroke (width 0) (type default) (color 0 0 0 0))
@@
     (property "Intersheet References" "${INTERSHEET_REFS}" (id 0) (at 178.8221 142.9544 0)
       (effects (font (size 1.27 1.27)) (justify left) hide)
-    )
-  )
-  (global_label "vccd" (shape input) (at 252.73 103.505 180) (fields_autoplaced)
-    (effects (font (size 1.27 1.27)) (justify right))
-    (property "Intersheet References" "${INTERSHEET_REFS}" (id 0) (at 210.82 -50.165 0)
-      (effects (font (size 1.27 1.27)) hide)
     )
   )
@@
     (pin "1")
   )
+  (symbol (lib_id "power:GND") (at 252.73 129.54 270) (mirror x) (unit 1)
+    (in_bom yes) (on_board yes)
+    (property "Reference" "#PWR?" (id 0) (at 246.38 129.54 0)
+      (effects (font (size 1.27 1.27)) hide)
+    )
+    (property "Value" "GND" (id 1) (at 247.65 129.54 90))
+    (property "Footprint" "" (id 2) (at 252.73 129.54 0)
+      (effects (font (size 1.27 1.27)) hide)
+    )
+    (property "Datasheet" "" (id 3) (at 252.73 129.54 0)
+      (effects (font (size 1.27 1.27)) hide)
+    )
+    (pin "1")
+  )
   (symbol (lib_id "power:GND") (at 92.71 38.1 180) (unit 1)
     (in_bom yes) (on_board yes)
@@
     (pin "1")
   )
+  (symbol (lib_id "power:GND") (at 252.73 103.505 270) (mirror x) (unit 1)
+    (in_bom yes) (on_board yes)
+    (property "Reference" "#PWR?" (id 0) (at 246.38 103.505 0)
+      (effects (font (size 1.27 1.27)) hide)
+    )
+    (property "Value" "GND" (id 1) (at 247.65 103.505 90))
+    (property "Footprint" "" (id 2) (at 252.73 103.505 0)
+      (effects (font (size 1.27 1.27)) hide)
+    )
+    (property "Datasheet" "" (id 3) (at 252.73 103.505 0)
+      (effects (font (size 1.27 1.27)) hide)
+    )
+    (pin "1")
+  )
   (symbol (lib_id "Device:C") (at 196.85 41.275 180) (unit 1)
     (in_bom yes) (on_board yes)
@@
     (pin "1")
     (pin "2")
+  )
+  (symbol (lib_id "power:GND") (at 252.73 132.08 270) (mirror x) (unit 1)
+    (in_bom yes) (on_board yes)
+    (property "Reference" "#PWR?" (id 0) (at 246.38 132.08 0)
+      (effects (font (size 1.27 1.27)) hide)
+    )
+    (property "Value" "GND" (id 1) (at 247.65 132.08 90))
+    (property "Footprint" "" (id 2) (at 252.73 132.08 0)
+      (effects (font (size 1.27 1.27)) hide)
+    )
+    (property "Datasheet" "" (id 3) (at 252.73 132.08 0)
+      (effects (font (size 1.27 1.27)) hide)
+    )
+    (pin "1")
   )
   (symbol (lib_id "power:GND") (at 121.285 132.715 0) (unit 1)
@@
     (pin "9")
   )
+  (symbol (lib_id "power:GND") (at 252.73 127 270) (mirror x) (unit 1)
+    (in_bom yes) (on_board yes)
+    (property "Reference" "#PWR?" (id 0) (at 246.38 127 0)
+      (effects (font (size 1.27 1.27)) hide)
+    )
+    (property "Value" "GND" (id 1) (at 247.65 127 90))
+    (property "Footprint" "" (id 2) (at 252.73 127 0)
+      (effects (font (size 1.27 1.27)) hide)
+    )
+    (property "Datasheet" "" (id 3) (at 252.73 127 0)
+      (effects (font (size 1.27 1.27)) hide)
+    )
+    (pin "1")
+  )
   (symbol (lib_id "power:GND") (at 140.97 69.85 90) (unit 1)
     (in_bom yes) (on_board yes)
@@
     (pin "9")
   )
+  (symbol (lib_id "power:GND") (at 252.73 119.38 270) (mirror x) (unit 1)
+    (in_bom yes) (on_board yes)
+    (property "Reference" "#PWR?" (id 0) (at 246.38 119.38 0)
+      (effects (font (size 1.27 1.27)) hide)
+    )
+    (property "Value" "GND" (id 1) (at 247.65 119.38 90))
+    (property "Footprint" "" (id 2) (at 252.73 119.38 0)
+      (effects (font (size 1.27 1.27)) hide)
+    )
+    (property "Datasheet" "" (id 3) (at 252.73 119.38 0)
+      (effects (font (size 1.27 1.27)) hide)
+    )
+    (pin "1")
+  )
   (symbol (lib_id "Device:R_US") (at 212.09 104.14 0) (unit 1)
     (in_bom yes) (on_board yes) (fields_autoplaced)
@@
     (pin "1")
   )
+  (symbol (lib_id "power:GND") (at 252.73 116.84 270) (mirror x) (unit 1)
+    (in_bom yes) (on_board yes)
+    (property "Reference" "#PWR?" (id 0) (at 246.38 116.84 0)
+      (effects (font (size 1.27 1.27)) hide)
+    )
+    (property "Value" "GND" (id 1) (at 247.65 116.84 90))
+    (property "Footprint" "" (id 2) (at 252.73 116.84 0)
+      (effects (font (size 1.27 1.27)) hide)
+    )
+    (property "Datasheet" "" (id 3) (at 252.73 116.84 0)
+      (effects (font (size 1.27 1.27)) hide)
+    )
+    (pin "1")
+  )
   (symbol (lib_id "power:GND") (at 154.305 132.715 0) (unit 1)
     (in_bom yes) (on_board yes)
@@
     )
     (property "Datasheet" "" (id 3) (at 265.43 90.805 0)
+      (effects (font (size 1.27 1.27)) hide)
+    )
+    (pin "1")
+  )
+  (symbol (lib_id "power:GND") (at 252.73 121.92 270) (mirror x) (unit 1)
+    (in_bom yes) (on_board yes)
+    (property "Reference" "#PWR?" (id 0) (at 246.38 121.92 0)
+      (effects (font (size 1.27 1.27)) hide)
+    )
+    (property "Value" "GND" (id 1) (at 247.65 121.92 90))
+    (property "Footprint" "" (id 2) (at 252.73 121.92 0)
+      (effects (font (size 1.27 1.27)) hide)
+    )
+    (property "Datasheet" "" (id 3) (at 252.73 121.92 0)
       (effects (font (size 1.27 1.27)) hide)
     )
@@
     (pin "1")
   )
+  (symbol (lib_id "power:GND") (at 252.73 124.46 270) (mirror x) (unit 1)
+    (in_bom yes) (on_board yes)
+    (property "Reference" "#PWR?" (id 0) (at 246.38 124.46 0)
+      (effects (font (size 1.27 1.27)) hide)
+    )
+    (property "Value" "GND" (id 1) (at 247.65 124.46 90))
+    (property "Footprint" "" (id 2) (at 252.73 124.46 0)
+      (effects (font (size 1.27 1.27)) hide)
+    )
+    (property "Datasheet" "" (id 3) (at 252.73 124.46 0)
+      (effects (font (size 1.27 1.27)) hide)
+    )
+    (pin "1")
+  )
   (symbol (lib_id "power:GND") (at 90.17 102.87 0) (unit 1)
     (in_bom yes) (on_board yes)
@@
       (reference "#PWR0101") (unit 1) (value "GND") (footprint "")
     )
+    (path "/2b5f1e97-25f1-479f-a1b3-fd02e7ef7f30"
+      (reference "#PWR?") (unit 1) (value "GND") (footprint "")
+    )
+    (path "/4dc92178-5bfc-4fc1-b2ec-ea248ef974f1"
+      (reference "#PWR?") (unit 1) (value "GND") (footprint "")
+    )
+    (path "/4fe9870f-7b73-42ce-933b-414a041b84b9"
+      (reference "#PWR?") (unit 1) (value "GND") (footprint "")
+    )
+    (path "/7d10675b-f02f-4c9d-b662-21f664b768c9"
+      (reference "#PWR?") (unit 1) (value "GND") (footprint "")
+    )
+    (path "/998a91f3-8485-4a91-bbfa-48e0f9c43bf7"
+      (reference "#PWR?") (unit 1) (value "GND") (footprint "")
+    )
+    (path "/b9d6b0a5-43d4-4f23-bd09-eb3b87073ac6"
+      (reference "#PWR?") (unit 1) (value "GND") (footprint "")
+    )
+    (path "/cf37dea4-dc69-4a76-a69e-17ea8a02cd6f"
+      (reference "#PWR?") (unit 1) (value "GND") (footprint "")
+    )
+    (path "/dae5ccaf-3843-4245-9bba-29652788e80d"
+      (reference "#PWR?") (unit 1) (value "GND") (footprint "")
+    )
     (path "/c7d3e54d-8b38-4424-8a5c-583eb3af3c03"
